File: midi-interface.kicad_pcb (KiCad board)
At the start: 2 copper layers, 55.9 x 73.7 mm, 20 parts, among them J1 MIDI-DIN-5, J2 MIDI-DIN-5, J3 MIDI-DIN-5, J4 Conn_01x05_Pin, U1 74HCT00, U3 H11L1

Commit message: Updated design
Parts:
- added H1: MountingHole_Pad, MountingHole:MountingHole_3.2mm_M3_ISO7380_Pad_TopBottom, F.Cu at (85.0, 20.0)
- added H2: MountingHole_Pad, MountingHole:MountingHole_3.2mm_M3_ISO7380_Pad_TopBottom, F.Cu at (130.0, 20.0)
- added H3: MountingHole_Pad, MountingHole:MountingHole_3.2mm_M3_ISO7380_Pad_TopBottom, F.Cu at (85.0, 97.5)
- added H4: MountingHole_Pad, MountingHole:MountingHole_3.2mm_M3_ISO7380_Pad_TopBottom, F.Cu at (130.0, 97.5)
Other:
- board size 55.9 x 73.7 mm -> 55.9 x 88.4 mm
