File: midi-interface.kicad_sch (KiCad schematic)
At the start: 20 parts, among them J1 MIDI-DIN-5, J2 MIDI-DIN-5, J3 MIDI-DIN-5, J4 Conn_01x05_Pin, U1 74HCT00, U3 H11L1

Commit message: Updated design
Parts:
- added H1, H2, H3, H4: MountingHole_Pad, symbol Mechanical:MountingHole_Pad
Connections:
- net GND: now also H1.1, H2.1, H3.1, H4.1

Commit message: Small update
Parts:
- H1, H2, H3, H4: footprint (none) -> MountingHole:MountingHole_3.2mm_M3_ISO7380_Pad_TopBottom
Changed lines of the file:
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@@
 			)
 		)
-		(property "Footprint" ""
+		(property "Footprint" "MountingHole:MountingHole_3.2mm_M3_ISO7380_Pad_TopBottom"
 			(at 260.35 36.83 0)
 			(effects
@@
 			)
 		)
-		(property "Footprint" ""
+		(property "Footprint" "MountingHole:MountingHole_3.2mm_M3_ISO7380_Pad_TopBottom"
 			(at 260.35 20.32 0)
 			(effects
@@
 			)
 		)
-		(property "Footprint" ""
+		(property "Footprint" "MountingHole:MountingHole_3.2mm_M3_ISO7380_Pad_TopBottom"
 			(at 260.35 69.85 0)
 			(effects
@@
 			)
 		)
-		(property "Footprint" ""
+		(property "Footprint" "MountingHole:MountingHole_3.2mm_M3_ISO7380_Pad_TopBottom"
 			(at 260.35 53.34 0)
 			(effects
